File: 03_Power/EPS_PCB/EPS_Bench2S_FlightLike/01_PV_Input.kicad_sch (KiCad schematic)
At the start: 7 parts

Commit message: EPS: lock unsafe KiCad placeholder
Other:
- note added: "NO FABRICAR: topología solar preliminar; entradas y ratings siguen TBD."
- note removed: "String A activo: P1 y P2 en serie. String B reservado (futuro)."
Changed lines of the file:
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@@
 		(title "01_PV_Input")
 	)
-	(text "String A activo: P1 y P2 en serie. String B reservado (futuro)."
+	(text "NO FABRICAR: topología solar preliminar; entradas y ratings siguen TBD."
 		(exclude_from_sim no)
 		(at 93.83 50.82 0)
@@
 		)
 		(stroke
-			(width 0.15)
-			(type solid)
-		)
-	)
-	(wire
-		(pts
-			(xy 188.83 93.82) (xy 188.83 106.82)
-		)
-		(stroke
