File: 03_Power/EPS_PCB/EPS_Bench2S_FlightLike/02_MPPT_Charger.kicad_sch (KiCad schematic)
At the start: 2 parts

Commit message: EPS: lock unsafe KiCad placeholder
Other:
- note added: "Entradas y salidas deliberadamente desconectadas hasta diseñar y revisar el circuito."
- note added: "NO FABRICAR: marcador de interfaz; no contiene MPPT ni cargador CC/CV."
- note removed: "Interfaz funcional: entrada PV y salida a BMS (Battery Management System)."
- note removed: "MPPT (Maximum Power Point Tracking) con módulo COTS (Commercial Off-The-Shelf) de banco."
Changed lines of the file:
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@@
 		(title "02_MPPT_Charger")
 	)
-	(text "MPPT (Maximum Power Point Tracking) con módulo COTS (Commercial Off-The-Shelf) de banco."
+	(text "NO FABRICAR: marcador de interfaz; no contiene MPPT ni cargador CC/CV."
 		(exclude_from_sim no)
 		(at 20 15 0)
@@
 		)
 	)
-	(text "Interfaz funcional: entrada PV y salida a BMS (Battery Management System)."
+	(text "Entradas y salidas deliberadamente desconectadas hasta diseñar y revisar el circuito."
 		(exclude_from_sim no)
 		(at 20 20 0)
@@
 		)
 	)
-	(wire
-		(pts
-			(xy 120 56) (xy 170 56)
-		)
-		(stroke
-			(width 0.15)
-			(type solid)
-		)
-	)
-	(wire
-		(pts
-			(xy 20 64) (xy 60 64)
-		)
-		(stroke
-			(width 0.15)
-			(type solid)
-		)
-	)
-	(wire
-		(pts
-			(xy 120 64) (xy 170 64)
-		)
-		(stroke
-			(width 0.15)
-			(type solid)
-		)
-	)
-	(wire
-		(pts
-			(xy 20 56) (xy 60 56)
-		)
-		(stroke
-			(width 0.15)
-			(type solid)
-		)
-	)
