File: 03_Power/EPS_PCB/EPS_Bench2S_FlightLike/03_Battery_BMS_2S.kicad_sch (KiCad schematic)
At the start: 3 parts

Commit message: EPS: lock unsafe KiCad placeholder
Other:
- note added: "NO FABRICAR: BMS, protecciones y pack 2S no están implementados."
- note added: "Pines de interfaz deliberadamente desconectados; no existe salida protegida."
- note removed: "BMS (Battery Management System) 2S de banco con pines funcionales B+, BM, B-."
- note removed: "Salida protegida del pack por BMS_P/BMS_N hacia bus VBAT."
Changed lines of the file:
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@@
 		(title "03_Battery_BMS_2S")
 	)
-	(text "Salida protegida del pack por BMS_P/BMS_N hacia bus VBAT."
+	(text "NO FABRICAR: BMS, protecciones y pack 2S no están implementados."
 		(exclude_from_sim no)
 		(at 20 20 0)
@@
 		)
 	)
-	(text "BMS (Battery Management System) 2S de banco con pines funcionales B+, BM, B-."
+	(text "Pines de interfaz deliberadamente desconectados; no existe salida protegida."
 		(exclude_from_sim no)
 		(at 20 15 0)
@@
 		)
 	)
-	(wire
-		(pts
-			(xy 20 64) (xy 180 64)
-		)
-		(stroke
-			(width 0.15)
-			(type solid)
-		)
-	)
-	(wire
-		(pts
-			(xy 20 56) (xy 180 56)
-		)
-		(stroke
-			(width 0.15)
-			(type solid)
-		)
-	)
-	(wire
-		(pts
-			(xy 65 72) (xy 180 72)
-		)
-		(stroke
-			(width 0.15)
-			(type solid)
-		)
-	)
