File: 03_Power/EPS_PCB/EPS_Bench2S_FlightLike/04_Power_Rails_5V_3V3.kicad_sch (KiCad schematic)
At the start: 2 parts

Commit message: EPS: lock unsafe KiCad placeholder
Other:
- note added: "Entradas/salidas deliberadamente desconectadas; corrientes objetivo TBD."
- note added: "NO FABRICAR: rails, regulación, límites y protecciones no están diseñados."
- note removed: "Módulos buck genéricos: VIN, GND, VOUT, EN."
- note removed: "Objetivos: +5V/2A y +3V3/1.5A."
Changed lines of the file:
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@@
 		(title "04_Power_Rails_5V_3V3")
 	)
-	(text "Objetivos: +5V/2A y +3V3/1.5A."
+	(text "NO FABRICAR: rails, regulación, límites y protecciones no están diseñados."
 		(exclude_from_sim no)
 		(at 20 20 0)
@@
 		)
 	)
-	(text "Módulos buck genéricos: VIN, GND, VOUT, EN."
+	(text "Entradas/salidas deliberadamente desconectadas; corrientes objetivo TBD."
 		(exclude_from_sim no)
 		(at 20 15 0)
@@
 		)
 	)
-	(wire
-		(pts
-			(xy 20 64) (xy 180 64)
-		)
-		(stroke
-			(width 0.15)
-			(type solid)
-		)
-	)
-	(wire
-		(pts
-			(xy 20 54) (xy 180 54)
-		)
-		(stroke
-			(width 0.15)
-			(type solid)
-		)
-	)
-	(wire
-		(pts
-			(xy 60 64) (xy 180 74)
-		)
-		(stroke
-			(width 0.15)
-			(type solid)
-		)
-	)
