File: 03_Power/EPS_PCB/EPS_Bench2S_FlightLike/05_Power_Gating.kicad_sch (KiCad schematic)
At the start: 2 parts

Commit message: EPS: lock unsafe KiCad placeholder
Other:
- note added: "NO FABRICAR: switches high-side y estados seguros no están diseñados."
- note removed: "Bloques de switch de carga: entrada, salida y enable."
Changed lines of the file:
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@@
 		(title "05_Power_Gating")
 	)
-	(text "Bloques de switch de carga: entrada, salida y enable."
+	(text "NO FABRICAR: switches high-side y estados seguros no están diseñados."
 		(exclude_from_sim no)
 		(at 20 15 0)
@@
 		)
 	)
-	(wire
-		(pts
-			(xy 20 62) (xy 180 62)
-		)
-		(stroke
-			(width 0.15)
-			(type solid)
-		)
-	)
-	(wire
-		(pts
-			(xy 60 70) (xy 180 70)
-		)
-		(stroke
-			(width 0.15)
-			(type solid)
-		)
-	)
-	(wire
-		(pts
-			(xy 130 78) (xy 180 78)
-		)
-		(stroke
-			(width 0.15)
-			(type solid)
-		)
-	)
-	(wire
-		(pts
-			(xy 20 52) (xy 180 52)
-		)
-		(stroke
-			(width 0.15)
-			(type solid)
-		)
-	)
 	(hierarchical_label "SW_5V_RF_EN"
-		(shape output)
+		(shape input)
 		(at 180 70 0)
 		(effects
@@
 	)
 	(hierarchical_label "SW_3V3_OBC_EN"
-		(shape output)
+		(shape input)
 		(at 180 78 0)
 		(effects
