File: 03_Power/EPS_PCB/EPS_Bench2S_FlightLike/06_Telemetry_TestPoints.kicad_sch (KiCad schematic)
At the start: 3 parts

Commit message: EPS: lock unsafe KiCad placeholder
Other:
- note added: "NO FABRICAR: telemetría y test points deliberadamente desconectados."
- note removed: "Breakouts INA219 con SDA, SCL, VIN+, VIN-."
Changed lines of the file:
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@@
 		(title "06_Telemetry_TestPoints")
 	)
-	(text "Breakouts INA219 con SDA, SCL, VIN+, VIN-."
+	(text "NO FABRICAR: telemetría y test points deliberadamente desconectados."
 		(exclude_from_sim no)
 		(at 20 15 0)
