File: 03_Power/EPS_PCB/EPS_Bench2S_FlightLike/EPS_Bench2S_FlightLike.kicad_sch (KiCad schematic)
At the start: 0 parts

Commit message: EPS: lock unsafe KiCad placeholder
Other:
- title: EPS Bench 2S Flight-Like -> EPS 2S NON-FABRICABLE PLACEHOLDER
Changed lines of the file:
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@@
 	(paper "A4")
 	(title_block
-		(title "EPS Bench 2S Flight-Like")
-		(comment 1 "Raíz del proyecto")
+		(title "EPS 2S NON-FABRICABLE PLACEHOLDER")
+		(comment 1 "NO FABRICAR / NO CONECTAR BATERIA")
 	)
 	(sheet
